File: pcb/si446x-dev.brd (EAGLE design)
At the start: 160 x 100 mm, 24 parts, among them U1 SI446X, X1 30 MHz

Commit message: Finish board
Parts:
- removed C9: 100pF, Capacitor:CAP0603
- removed TP1, TP2, TP3, TP4, TP5: TESTPOINT, PADs:PAD1.27MM
- added JP1, JP2: PINHD-1X8, Pin Header:1X08
- added L8: 12nH, Inductor:IND0603
- added LOGO1: OSHW-LOGOM, Silkscreen:OSHW-LOGO-M
- C1: value 1.2pF -> 1uF
- C2: value 3pF -> 100nF
- C3: value 5.1pF -> 100pF
- C4: value 6.8nH -> 5.1pF
- C5: value 3.3pF -> 3pF
- C6: value 3.3pF -> 1.2pF
- C7: value 1uF -> 3.3pF
- C8: value 100nF -> 3.3pF
- L2: value 3.3nH -> 18nH
- L3: value 12nH -> 3.3nH
- L5: value 12nH -> 6.8nH
- L6: value 18nH -> 12nH
- moved RFCON1 52.0 mm to (20.2, 23.5), turned to 180 degrees
- moved C6 46.0 mm to (15.2, 16.0), turned to 90 degrees
- moved L2 42.3 mm to (14.2, 13.4), turned to 180 degrees
- moved X1 41.8 mm to (17.4, 5.70), turned to 270 degrees
- moved C2 39.1 mm to (5.40, 9.20), turned to 270 degrees
- moved C5 37.7 mm to (11.6, 14.2), turned to 90 degrees
- moved L5 37.3 mm to (8.30, 20.1)
- moved L4 35.3 mm to (13.4, 16.0), turned to 90 degrees
- moved C8 34.5 mm to (14.2, 26.1), turned to 90 degrees
- moved L7 34.0 mm to (11.7, 23.5)
- moved C1 33.6 mm to (5.40, 12.6), turned to 90 degrees
- moved C4 30.3 mm to (9.10, 14.2), turned to 90 degrees
- moved L1 29.3 mm to (7.20, 12.6), turned to 90 degrees
- moved U1 27.6 mm to (12.1, 9.00), turned to 270 degrees
- moved C7 26.1 mm to (10.9, 26.1), turned to 90 degrees
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Connections:
- removed net N$11: TP4.TP, U1.20
- removed net N$12: TP3.TP, U1.19
- removed net N$13: TP2.TP, U1.10
- removed net N$14: TP1.TP, U1.9
- new net !CS: JP1.2, U1.15
- new net !IRQ: JP1.6, U1.11
- new net EN: JP2.6, U1.1
- new net IO0: JP2.2, U1.9
- new net IO1: JP2.3, U1.10
- new net IO2: JP2.4, U1.19
- new net IO3: JP2.5, U1.20
- new net MISO: JP1.4, U1.13
- new net MOSI: JP1.3, U1.14
- new net SCK: JP1.5, U1.12
- net 3V3: now also C1.1, C2.1, C3.1, JP1.1, JP2.1; no longer C7.1, C8.1, C9.1
- net GND: now also C1.2, C3.2, JP1.7, JP1.8, JP2.7, JP2.8, L5.1; no longer C4.2, C6.2, C9.2, TP5.TP
- net N$1: now also C5.1, L2.2, L4.1; no longer C2.1, L6.2, L7.1
- net N$2: now also C6.1, L2.1; no longer C1.1, L6.1
- net N$3: now also C6.2, L3.2, L4.2, L5.2, L6.1; no longer C1.2, C4.1, L2.2, L3.1, L7.2
- net N$4: now also L8.2; no longer L5.2
- net N$5: now also C4.2, L3.1; no longer C3.2, L2.1
- net N$6: now also C4.1; no longer C3.1
- net N$7: now also C7.1, L6.2, L7.1; no longer C5.1, L3.2, L4.1
- net N$8: now also C8.1, L7.2, L8.1; no longer C6.1, L4.2, L5.1
Routing:
- net 3V3: track 0.00 -> 45.7 mm, vias 0 -> 2
- net IO0: track 0.00 -> 17.7 mm, vias 0 -> 1
- net !IRQ: track 0.00 -> 17.2 mm, vias 0 -> 1
- net SCK: track 0.00 -> 16.3 mm, vias 0 -> 1
- net !CS: track 0.00 -> 15.7 mm, vias 0 -> 1
- net MISO: track 0.00 -> 15.3 mm, vias 0 -> 1
- net MOSI: track 0.00 -> 14.5 mm, vias 0 -> 1
- net IO1: track 0.00 -> 14.4 mm, vias 0 -> 1
- net N$3: track 0.00 -> 11.5 mm
- net EN: track 0.00 -> 10.3 mm
- net IO3: track 0.00 -> 8.67 mm
- net IO2: track 0.00 -> 8.21 mm
- net N$1: track 0.00 -> 6.63 mm
- net N$6: track 0.00 -> 6.15 mm
- net N$2: track 0.00 -> 5.97 mm
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- added copper zone on layer 1, net GND
- added copper zone on layer 16, net GND
Other:
- board size 160 x 100 mm -> 23.9 x 28.5 mm
- board text added: "GND GND !IRQ! SCK MISO MOSI !CS! 3V3"
- board text added: "GND GND EN IO3 IO2 IO1 IO0 3V3"
