File: pcb/si446x-dev.brd (EAGLE design)
At the start: 23.9 x 28.5 mm, 22 parts, among them U1 SI446X, X1 30 MHz

Commit message: Update libs
Parts:
- U1: value SI446X -> SI4463
Changed lines of the file:
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@@
 <?xml version="1.0" encoding="utf-8"?>
 <!DOCTYPE eagle SYSTEM "eagle.dtd">
-<eagle version="9.3.0">
+<eagle version="9.3.2">
 <drawing>
 <settings>
-<setting alwaysvectorfont="yes"/>
+<setting alwaysvectorfont="no"/>
 <setting verticaltext="up"/>
 </settings>
@@
 </element>
 <element name="RFCON1" library="RF Connector" package="U.FL" value="RFCON-U.FL" x="20.2" y="23.5" smashed="yes" rot="R180"/>
-<element name="U1" library="Silicon Labs" package="QFN20" value="SI446X" x="12.1" y="9" smashed="yes" rot="R270">
+<element name="U1" library="Silicon Labs" package="QFN20" value="SI4463" x="12.1" y="9" smashed="yes" rot="R270">
 <attribute name="NAME" x="10.1" y="5.419" size="0.762" layer="25" font="vector" ratio="10"/>
 </element>
