File: pcb/si446x-dev.sch (EAGLE design)
At the start: 24 parts, among them U1 SI446X, X1 30 MHz

Commit message: Finish board
Parts:
- removed C9: 100pF, Capacitor:CAPACITOR-0603
- removed TP1, TP2, TP3, TP4, TP5: TESTPOINT, PADs:TESTPOINT
- added JP1, JP2: PINHD-1X8, Pin Header:PINHD-1X8
- added L8: 12nH, Inductor:INDUCTOR-0603
- added LOGO1: OSHW-LOGOM, Silkscreen:OSHW-LOGOM
- C1: value 1.2pF -> 1uF
- C2: value 3pF -> 100nF
- C3: value 5.1pF -> 100pF
- C4: value 6.8nH -> 5.1pF
- C5: value 3.3pF -> 3pF
- C6: value 3.3pF -> 1.2pF
- C7: value 1uF -> 3.3pF
- C8: value 100nF -> 3.3pF
- L2: value 3.3nH -> 18nH
- L3: value 12nH -> 3.3nH
- L5: value 12nH -> 6.8nH
- L6: value 18nH -> 12nH
Connections:
- removed net N$11: TP4.TP, U1.GPIO3
- removed net N$12: TP3.TP, U1.GPIO2
- removed net N$13: TP2.TP, U1.GPIO1
- removed net N$14: TP1.TP, U1.GPIO0
- new net !CS: JP1-2.S, U1.!SEL
- new net !IRQ: JP1-6.S, U1.!IRQ
- new net EN: JP2-6.S, U1.SDN
- new net IO0: JP2-2.S, U1.GPIO0
- new net IO1: JP2-3.S, U1.GPIO1
- new net IO2: JP2-4.S, U1.GPIO2
- new net IO3: JP2-5.S, U1.GPIO3
- new net MISO: JP1-4.S, U1.SDO
- new net MOSI: JP1-3.S, U1.SDI
- new net SCK: JP1-5.S, U1.SCLK
- net 3V3: now also C1.C1, C2.C1, C3.C1, JP1-1.S, JP2-1.S; no longer C7.C1, C8.C1, C9.C1
- net GND: now also C1.C2, C3.C2, JP1-7.S, JP1-8.S, JP2-7.S, JP2-8.S, L5.1; no longer C4.C2, C6.C2, C9.C2, TP5.TP
- net N$1: now also C5.C1, L2.2, L4.1; no longer C2.C1, L6.2, L7.1
- net N$2: now also C6.C1, L2.1; no longer C1.C1, L6.1
- net N$3: now also C6.C2, L3.2, L4.2, L5.2, L6.1; no longer C1.C2, C4.C1, L2.2, L3.1, L7.2
- net N$4: now also L8.2; no longer L5.2
- net N$5: now also C4.C2, L3.1; no longer C3.C2, L2.1
- net N$6: now also C4.C1; no longer C3.C1
- net N$7: now also C7.C1, L6.2, L7.1; no longer C5.C1, L3.2, L4.1
- net N$8: now also C8.C1, L7.2, L8.1; no longer C6.C1, L4.2, L5.1
Other:
- moved on the sheet: C1, C2, C3, C4, C5, C6, C7, C8, L2, L3, L4, L5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

Commit message: Update libs
Parts:
- U1: value SI446X -> SI4463; device Silicon Labs:SI446X -> Silicon Labs:SI4463
Changed lines of the file:
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@@
 <?xml version="1.0" encoding="utf-8"?>
 <!DOCTYPE eagle SYSTEM "eagle.dtd">
-<eagle version="9.3.0">
+<eagle version="9.3.2">
 <drawing>
 <settings>
@@
 <attribute name="DESIGNER" value=""/>
 </part>
-<part name="U1" library="Silicon Labs" deviceset="SI446X" device=""/>
+<part name="U1" library="Silicon Labs" deviceset="SI446*" device="" technology="3"/>
 <part name="L1" library="Inductor" deviceset="INDUCTOR" device="-0603" value="120nH"/>
 <part name="L3" library="Inductor" deviceset="INDUCTOR" device="-0603" value="3.3nH"/>
